File: hardware/floppy-adapter/floppy-adapter.kicad_sch (KiCad schematic)
At the start: 12 parts, among them J1 Conn_02x17 socket (O1 side), J2 Conn_02x17 header (OEM cable), J3 Conn_02x17 header (Gotek), J4 Gotek power, J5 Panel switch, K1 4PDT relay, 5V coil

Commit message: hardware: pass TG43/EARLY through on the floppy adapter, not to GND (#62)
Reading the mainboard schematic itself (DWG 1A2011-00 Rev E, sheet 9 of 9,
DISC CONTROLLER) rather than the drive-side drawing shows P8 pin 4 = TG43 and
pin 6 = EARLY, both driven by the FDC through 7406 open-collector buffers, with
GND = 1,2,3,5,9,19,27,29,31,33. The archived Visser adapter that the pin table
was transcribed from ties 2, 4, 6 and 7 to GND. That is harmless for a
Gotek-only adapter, but this card switches the OEM cable through to the
physical drives, and TG43 is the drive's write-current-reduce input on 96 tpi
drives, so clamping it low would assert reduced write current permanently.

Pins 4 and 6 now carry FLP_TG43 / FLP_EARLY and pass straight through J1 -> J2.
Pins 2 and 7 stay on GND: the mainboard drawing grounds pin 2 and the drive-end
drawing (1A3004 P2) grounds pin 7, and neither is a driven signal, so tying
both is safe whichever drawing is right.

docs/floppy-adapter-design.md section 2's table and citation are corrected with
it - it cited DWG 1A3004, the disk-electronics drawing, for a fact that lives
on 1A2011-00. tools/check_schematics.py still passes: 24 nets, ERC 0 errors.

part of #62
Connections:
- net GND: no longer J1.4 (GND), J1.6 (GND), J2.4 (GND), J2.6 (GND)
- new net FLP_EARLY: J1.6 (EARLY), J2.6 (EARLY)
- new net FLP_TG43: J1.4 (TG43), J2.4 (TG43)
Changed lines of the file:
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@@
   (label "GND" (at 71.12 40.63999999999999 0) (effects (font (size 1.27 1.27)) (justify left bottom)))
   (label "GND" (at 71.12 43.18 0) (effects (font (size 1.27 1.27)) (justify left bottom)))
-  (label "GND" (at 71.12 45.71999999999999 0) (effects (font (size 1.27 1.27)) (justify left bottom)))
+  (label "FLP_TG43" (at 71.12 45.71999999999999 0) (effects (font (size 1.27 1.27)) (justify left bottom)))
   (label "GND" (at 71.12 48.26 0) (effects (font (size 1.27 1.27)) (justify left bottom)))
-  (label "GND" (at 71.12 50.79999999999999 0) (effects (font (size 1.27 1.27)) (justify left bottom)))
+  (label "FLP_EARLY" (at 71.12 50.79999999999999 0) (effects (font (size 1.27 1.27)) (justify left bottom)))
   (label "GND" (at 71.12 53.339999999999996 0) (effects (font (size 1.27 1.27)) (justify left bottom)))
   (label "FLP_INDEX" (at 71.12 55.87999999999999 0) (effects (font (size 1.27 1.27)) (justify left bottom)))
@@
   (label "GND" (at 180.34 40.63999999999999 0) (effects (font (size 1.27 1.27)) (justify left bottom)))
   (label "GND" (at 180.34 43.18 0) (effects (font (size 1.27 1.27)) (justify left bottom)))
-  (label "GND" (at 180.34 45.71999999999999 0) (effects (font (size 1.27 1.27)) (justify left bottom)))
+  (label "FLP_TG43" (at 180.34 45.71999999999999 0) (effects (font (size 1.27 1.27)) (justify left bottom)))
   (label "GND" (at 180.34 48.26 0) (effects (font (size 1.27 1.27)) (justify left bottom)))
-  (label "GND" (at 180.34 50.79999999999999 0) (effects (font (size 1.27 1.27)) (justify left bottom)))
+  (label "FLP_EARLY" (at 180.34 50.79999999999999 0) (effects (font (size 1.27 1.27)) (justify left bottom)))
   (label "GND" (at 180.34 53.339999999999996 0) (effects (font (size 1.27 1.27)) (justify left bottom)))
   (label "FLP_INDEX" (at 180.34 55.87999999999999 0) (effects (font (size 1.27 1.27)) (justify left bottom)))
